Commit message: added frame for 3DOf to urdf

File: deltax_descriptions/urdf/deltaxs_v5_d800.urdf (robot description, URDF)
Before this commit: robot deltax_descriptions, 17 links, 16 joints
Links:
- added link 3_dof_frame
Joints:
- added joint 3_dof_frame_joint: type fixed, parent ball_moving_Link, child 3_dof_frame, origin xyz=0.0333733971724094 0.034641 0 rpy=0 0 0
