Commit message: new stls and various changes to URDF

File: deltax_descriptions/urdf/deltaxs_v5_d800.urdf.xacro (robot description, xacro)
@@ -1,7 +1,4 @@
 <?xml version="1.0" encoding="utf-8"?>
-<!-- This URDF was automatically created by SolidWorks to URDF Exporter! Originally created by Stephen Brawner (brawner@gmail.com)
-     Commit Version: 1.6.0-1-g15f4949  Build Version: 1.6.7594.29634
-     For more information. please see http://wiki.ros.org/sw_urdf_exporter -->
-<robot name="deltax_descriptions">
+<robot xmlns:xacro="http://wiki.ros.org/xacro" name="deltax_d800">
 <!-- Serial Chain -->
   <link name="base_link">
@@ -212,5 +209,6 @@
   <link name="axis6_link">
     <visual>
-      <origin xyz="-0.014 0 0.00268" rpy="1.57 0 3.14" />
+      <origin xyz="-0.014 0 -0.00268" rpy="-1.57 0 3.14" />
+      <!-- <origin xyz="-0.014 0 0.00268" rpy="1.57 0 3.14" /> -->
       <geometry>
         <mesh filename="package://deltax_descriptions/meshes/axis6_origin.STL" />
@@ -222,5 +220,5 @@
   </link>
   <joint name="theta5" type="revolute">
-    <origin xyz="0 0 -0.086" rpy="1.57 0 0" />
+    <origin xyz="0 0 -0.086" rpy="-1.57 0 0" />
     <parent link="axis5_link" />
     <child link="axis6_link" />
@@ -230,8 +228,7 @@
   <link name="axis6_flange_link">
     <visual>
-      <origin xyz="0 0 -0.01" rpy="0 0 0" />
-      <geometry>
-        <cylinder length="0.02" radius="0.0225" />
-        <mesh filename="package://deltax_descriptions/meshes/axis6_flange.STL" />
+      <origin xyz="0 0 0" rpy="0 1.57 0" />
+      <geometry>
+        <mesh filename="package://deltax_descriptions/meshes/axis6_flange_origin.STL" />
       </geometry>
       <material name="LightGrey">
@@ -241,5 +238,5 @@
   </link>
   <joint name="theta6" type="revolute">
-    <origin xyz="0 0 -0.026" rpy="0 1.57 0" />
+    <origin xyz="0 0 ${0.026-0.00268}" rpy="0 1.57 0" />
     <parent link="axis6_link" />
     <child link="axis6_flange_link" />

Commit message: recorded video and sharing for feedback

File: deltax_descriptions/urdf/deltaxs_v5_d800.urdf.xacro (robot description, xacro)
@@ -1,5 +1,10 @@
 <?xml version="1.0" encoding="utf-8"?>
 <robot xmlns:xacro="http://wiki.ros.org/xacro" name="deltax_d800">
-<!-- Serial Chain -->
+<!-- Materials - START -->
+  <material name="LightGrey">
+    <color rgba="0.792156862745098 0.819607843137255 0.933333333333333 1" />
+  </material>
+<!-- Materials - END -->
+<!-- Serial Chain - START -->
   <link name="base_link">
     <inertial>
@@ -35,7 +40,5 @@
         <mesh filename="package://deltax_descriptions/meshes/rf1_Link.STL" />
       </geometry>
-      <material name="LightGrey">
-        <color rgba="0.792156862745098 0.819607843137255 0.933333333333333 1" />
-      </material>
+      <material name="LightGrey"/>
     </visual>
     <collision>
@@ -63,7 +66,5 @@
         <mesh filename="package://deltax_descriptions/meshes/ball_top1_Link.STL" />
       </geometry>
-      <material name="LightGrey">
-        <color rgba="0.792156862745098 0.819607843137255 0.933333333333333 1" />
-      </material>
+      <material name="LightGrey"/>
     </visual>
     <collision>
@@ -91,7 +92,5 @@
         <mesh filename="package://deltax_descriptions/meshes/re1_Link.STL" />
       </geometry>
-      <material name="LightGrey">
-        <color rgba="0.792156862745098 0.819607843137255 0.933333333333333 1" />
-      </material>
+      <material name="LightGrey"/>
     </visual>
     <collision>
@@ -119,7 +118,5 @@
         <mesh filename="package://deltax_descriptions/meshes/ball_bot1_Link.STL" />
       </geometry>
-      <material name="LightGrey">
-        <color rgba="0.792156862745098 0.819607843137255 0.933333333333333 1" />
-      </material>
+      <material name="LightGrey"/>
     </visual>
     <collision>
@@ -147,7 +144,5 @@
         <mesh filename="package://deltax_descriptions/meshes/ball_moving_Link.STL" />
       </geometry>
-      <material name="LightGrey">
-        <color rgba="0.792156862745098 0.819607843137255 0.933333333333333 1" />
-      </material>
+      <material name="LightGrey"/>
     </visual>
     <collision>
@@ -164,5 +159,5 @@
     <axis xyz="-1 0 0" />
   </joint>
-<!-- New Links/Joints -->
+<!-- New Links/Joints - PLEASE REVIEW -->
   <link name="3_dof_frame"/>
   <joint name="3_dof_frame_joint" type="fixed">
@@ -177,7 +172,5 @@
         <mesh filename="package://deltax_descriptions/meshes/axis4_origin.STL" />
       </geometry>
-      <material name="LightGrey">
-        <color rgba="0.792156862745098 0.819607843137255 0.933333333333333 1" />
-      </material>
+      <material name="LightGrey"/>
     </visual>
   </link>
@@ -193,13 +186,9 @@
       <origin xyz="0 0 0" rpy="0 0 0" />
       <geometry>
-        <!-- <cylinder length="0.02" radius="0.03" /> -->
         <mesh filename="package://deltax_descriptions/meshes/axis5_origin.STL" />
       </geometry>
-      <material name="LightGrey">
-        <color rgba="0.792156862745098 0.819607843137255 0.933333333333333 1" />
-      </material>
-    </visual>
-  </link>
-<!-- TODO get correct xy(z) transform -->
+      <material name="LightGrey"/>
+    </visual>
+  </link>
   <joint name="fixed5" type="fixed">
     <origin xyz="0 0 -0.01" rpy="0 0 0" />
@@ -210,11 +199,8 @@
     <visual>
       <origin xyz="-0.014 0 -0.00268" rpy="-1.57 0 3.14" />
-      <!-- <origin xyz="-0.014 0 0.00268" rpy="1.57 0 3.14" /> -->
       <geometry>
         <mesh filename="package://deltax_descriptions/meshes/axis6_origin.STL" />
       </geometry>
-      <material name="LightGrey">
-        <color rgba="0.792156862745098 0.819607843137255 0.933333333333333 1" />
-      </material>
+      <material name="LightGrey"/>
     </visual>
   </link>
@@ -232,7 +218,5 @@
         <mesh filename="package://deltax_descriptions/meshes/axis6_flange_origin.STL" />
       </geometry>
-      <material name="LightGrey">
-        <color rgba="0.792156862745098 0.819607843137255 0.933333333333333 1" />
-      </material>
+      <material name="LightGrey"/>
     </visual>
   </link>
@@ -244,5 +228,6 @@
     <limit lower="-3.14" upper="3.14" effort="5.0" velocity="10.0"/>
   </joint>
-<!-- Fixed Links on Moving Platform -->
+<!-- Serial Chain - END -->
+<!-- Fixed Links on Moving Platform - START -->
   <link name="ball_bot2_Link">
     <inertial>
@@ -256,7 +241,5 @@
         <mesh filename="package://deltax_descriptions/meshes/ball_bot2_Link.STL" />
       </geometry>
-      <material name="LightGrey">
-        <color rgba="0.792156862745098 0.819607843137255 0.933333333333333 1" />
-      </material>
+      <material name="LightGrey"/>
     </visual>
     <collision>
@@ -284,7 +267,5 @@
         <mesh filename="package://deltax_descriptions/meshes/ball_bot3_Link.STL" />
       </geometry>
-      <material name="LightGrey">
-        <color rgba="0.792156862745098 0.819607843137255 0.933333333333333 1" />
-      </material>
+      <material name="LightGrey"/>
     </visual>
     <collision>
@@ -301,5 +282,6 @@
     <axis xyz="0 0 0" />
   </joint>
-<!-- Driven Parrallel Links -->
+<!-- Fixed Links on Moving Platform - END -->
+<!-- Driven Parallel Links - START -->
   <link name="re2_Link">
     <inertial>
@@ -313,7 +295,5 @@
         <mesh filename="package://deltax_descriptions/meshes/re2_Link.STL" />
       </geometry>
-      <material name="LightGrey">
-        <color rgba="0.792156862745098 0.819607843137255 0.933333333333333 1" />
-      </material>
+      <material name="LightGrey"/>
     </visual>
     <collision>
@@ -341,7 +321,5 @@
         <mesh filename="package://deltax_descriptions/meshes/rf2_Link.STL" />
       </geometry>
-      <material name="LightGrey">
-        <color rgba="0.792156862745098 0.819607843137255 0.933333333333333 1" />
-      </material>
+      <material name="LightGrey"/>
     </visual>
     <collision>
@@ -369,7 +347,5 @@
         <mesh filename="package://deltax_descriptions/meshes/ball_top2_Link.STL" />
       </geometry>
-      <material name="LightGrey">
-        <color rgba="0.792156862745098 0.819607843137255 0.933333333333333 1" />
-      </material>
+      <material name="LightGrey"/>
     </visual>
     <collision>
@@ -397,7 +373,5 @@
         <mesh filename="package://deltax_descriptions/meshes/re3_Link.STL" />
       </geometry>
-      <material name="LightGrey">
-        <color rgba="0.792156862745098 0.819607843137255 0.933333333333333 1" />
-      </material>
+      <material name="LightGrey"/>
     </visual>
     <collision>
@@ -425,7 +399,5 @@
         <mesh filename="package://deltax_descriptions/meshes/re4_Link.STL" />
       </geometry>
-      <material name="LightGrey">
-        <color rgba="0.792156862745098 0.819607843137255 0.933333333333333 1" />
-      </material>
+      <material name="LightGrey"/>
     </visual>
     <collision>
@@ -481,7 +453,5 @@
         <mesh filename="package://deltax_descriptions/meshes/ball_top3_Link.STL" />
       </geometry>
-      <material name="LightGrey">
-        <color rgba="0.792156862745098 0.819607843137255 0.933333333333333 1" />
-      </material>
+      <material name="LightGrey"/>
     </visual>
     <collision>
@@ -509,7 +479,5 @@
         <mesh filename="package://deltax_descriptions/meshes/re5_Link.STL" />
       </geometry>
-      <material name="LightGrey">
-        <color rgba="0.792156862745098 0.819607843137255 0.933333333333333 1" />
-      </material>
+      <material name="LightGrey"/>
     </visual>
     <collision>
@@ -537,7 +505,5 @@
         <mesh filename="package://deltax_descriptions/meshes/re6_Link.STL" />
       </geometry>
-      <material name="LightGrey">
-        <color rgba="0.792156862745098 0.819607843137255 0.933333333333333 1" />
-      </material>
+      <material name="LightGrey"/>
     </visual>
     <collision>
@@ -554,3 +520,4 @@
     <axis xyz="1 0 0" />
   </joint>
+<!-- Driven Parallel Links - END -->
 </robot>
