Commit message: ok working now, saving before adding 6 dof to driver

File: deltax_descriptions/urdf/deltaxs_v5_d800.urdf.xacro (robot description, xacro)
@@ -16,5 +16,5 @@
       <origin xyz="0 0 0" rpy="0 0 0" />
       <geometry>
-        <mesh filename="package://deltax_descriptions/meshes/base_link.STL" />
+        <mesh filename="package://deltax_descriptions/meshes/4_dof/base_link.STL" />
       </geometry>
       <material name="LightGrey">
@@ -25,5 +25,5 @@
       <origin xyz="0 0 0" rpy="0 0 0" />
       <geometry>
-        <mesh filename="package://deltax_descriptions/meshes/base_link.STL" />
+        <mesh filename="package://deltax_descriptions/meshes/4_dof/base_link.STL" />
       </geometry>
     </collision>
@@ -38,12 +38,12 @@
       <origin xyz="0 0 0" rpy="0 0 0" />
       <geometry>
-        <mesh filename="package://deltax_descriptions/meshes/rf1_Link.STL" />
-      </geometry>
-      <material name="LightGrey"/>
-    </visual>
-    <collision>
-      <origin xyz="0 0 0" rpy="0 0 0" />
-      <geometry>
-        <mesh filename="package://deltax_descriptions/meshes/rf1_Link.STL" />
+        <mesh filename="package://deltax_descriptions/meshes/4_dof/rf1_Link.STL" />
+      </geometry>
+      <material name="LightGrey"/>
+    </visual>
+    <collision>
+      <origin xyz="0 0 0" rpy="0 0 0" />
+      <geometry>
+        <mesh filename="package://deltax_descriptions/meshes/4_dof/rf1_Link.STL" />
       </geometry>
     </collision>
@@ -64,12 +64,12 @@
       <origin xyz="0 0 0" rpy="0 0 0" />
       <geometry>
-        <mesh filename="package://deltax_descriptions/meshes/ball_top1_Link.STL" />
-      </geometry>
-      <material name="LightGrey"/>
-    </visual>
-    <collision>
-      <origin xyz="0 0 0" rpy="0 0 0" />
-      <geometry>
-        <mesh filename="package://deltax_descriptions/meshes/ball_top1_Link.STL" />
+        <mesh filename="package://deltax_descriptions/meshes/4_dof/ball_top1_Link.STL" />
+      </geometry>
+      <material name="LightGrey"/>
+    </visual>
+    <collision>
+      <origin xyz="0 0 0" rpy="0 0 0" />
+      <geometry>
+        <mesh filename="package://deltax_descriptions/meshes/4_dof/ball_top1_Link.STL" />
       </geometry>
     </collision>
@@ -90,12 +90,12 @@
       <origin xyz="0 0 0" rpy="0 0 0" />
       <geometry>
-        <mesh filename="package://deltax_descriptions/meshes/re1_Link.STL" />
-      </geometry>
-      <material name="LightGrey"/>
-    </visual>
-    <collision>
-      <origin xyz="0 0 0" rpy="0 0 0" />
-      <geometry>
-        <mesh filename="package://deltax_descriptions/meshes/re1_Link.STL" />
+        <mesh filename="package://deltax_descriptions/meshes/4_dof/re1_Link.STL" />
+      </geometry>
+      <material name="LightGrey"/>
+    </visual>
+    <collision>
+      <origin xyz="0 0 0" rpy="0 0 0" />
+      <geometry>
+        <mesh filename="package://deltax_descriptions/meshes/4_dof/re1_Link.STL" />
       </geometry>
     </collision>
@@ -116,12 +116,12 @@
       <origin xyz="0 0 0" rpy="0 0 0" />
       <geometry>
-        <mesh filename="package://deltax_descriptions/meshes/ball_bot1_Link.STL" />
-      </geometry>
-      <material name="LightGrey"/>
-    </visual>
-    <collision>
-      <origin xyz="0 0 0" rpy="0 0 0" />
-      <geometry>
-        <mesh filename="package://deltax_descriptions/meshes/ball_bot1_Link.STL" />
+        <mesh filename="package://deltax_descriptions/meshes/4_dof/ball_bot1_Link.STL" />
+      </geometry>
+      <material name="LightGrey"/>
+    </visual>
+    <collision>
+      <origin xyz="0 0 0" rpy="0 0 0" />
+      <geometry>
+        <mesh filename="package://deltax_descriptions/meshes/4_dof/ball_bot1_Link.STL" />
       </geometry>
     </collision>
@@ -142,12 +142,12 @@
       <origin xyz="0 0 0" rpy="0 0 0" />
       <geometry>
-        <mesh filename="package://deltax_descriptions/meshes/ball_moving_Link.STL" />
-      </geometry>
-      <material name="LightGrey"/>
-    </visual>
-    <collision>
-      <origin xyz="0 0 0" rpy="0 0 0" />
-      <geometry>
-        <mesh filename="package://deltax_descriptions/meshes/ball_moving_Link.STL" />
+        <mesh filename="package://deltax_descriptions/meshes/4_dof/ball_moving_Link.STL" />
+      </geometry>
+      <material name="LightGrey"/>
+    </visual>
+    <collision>
+      <origin xyz="0 0 0" rpy="0 0 0" />
+      <geometry>
+        <mesh filename="package://deltax_descriptions/meshes/4_dof/ball_moving_Link.STL" />
       </geometry>
     </collision>
@@ -170,5 +170,5 @@
       <origin xyz="0 0 -0.01" rpy="0 0 0" />
       <geometry>
-        <mesh filename="package://deltax_descriptions/meshes/axis4_origin.STL" />
+        <mesh filename="package://deltax_descriptions/meshes/4_dof/axis4_origin.STL" />
       </geometry>
       <material name="LightGrey"/>
@@ -186,5 +186,5 @@
       <origin xyz="0 0 0" rpy="0 0 0" />
       <geometry>
-        <mesh filename="package://deltax_descriptions/meshes/axis5_origin.STL" />
+        <mesh filename="package://deltax_descriptions/meshes/4_dof/axis5_origin.STL" />
       </geometry>
       <material name="LightGrey"/>
@@ -200,5 +200,5 @@
       <origin xyz="-0.014 0 -0.00268" rpy="-1.57 0 3.14" />
       <geometry>
-        <mesh filename="package://deltax_descriptions/meshes/axis6_origin.STL" />
+        <mesh filename="package://deltax_descriptions/meshes/4_dof/axis6_origin.STL" />
       </geometry>
       <material name="LightGrey"/>
@@ -216,5 +216,5 @@
       <origin xyz="0 0 0" rpy="0 1.57 0" />
       <geometry>
-        <mesh filename="package://deltax_descriptions/meshes/axis6_flange_origin.STL" />
+        <mesh filename="package://deltax_descriptions/meshes/4_dof/axis6_flange_origin.STL" />
       </geometry>
       <material name="LightGrey"/>
@@ -239,12 +239,12 @@
       <origin xyz="0 0 0" rpy="0 0 0" />
       <geometry>
-        <mesh filename="package://deltax_descriptions/meshes/ball_bot2_Link.STL" />
-      </geometry>
-      <material name="LightGrey"/>
-    </visual>
-    <collision>
-      <origin xyz="0 0 0" rpy="0 0 0" />
-      <geometry>
-        <mesh filename="package://deltax_descriptions/meshes/ball_bot2_Link.STL" />
+        <mesh filename="package://deltax_descriptions/meshes/4_dof/ball_bot2_Link.STL" />
+      </geometry>
+      <material name="LightGrey"/>
+    </visual>
+    <collision>
+      <origin xyz="0 0 0" rpy="0 0 0" />
+      <geometry>
+        <mesh filename="package://deltax_descriptions/meshes/4_dof/ball_bot2_Link.STL" />
       </geometry>
     </collision>
@@ -265,12 +265,12 @@
       <origin xyz="0 0 0" rpy="0 0 0" />
       <geometry>
-        <mesh filename="package://deltax_descriptions/meshes/ball_bot3_Link.STL" />
-      </geometry>
-      <material name="LightGrey"/>
-    </visual>
-    <collision>
-      <origin xyz="0 0 0" rpy="0 0 0" />
-      <geometry>
-        <mesh filename="package://deltax_descriptions/meshes/ball_bot3_Link.STL" />
+        <mesh filename="package://deltax_descriptions/meshes/4_dof/ball_bot3_Link.STL" />
+      </geometry>
+      <material name="LightGrey"/>
+    </visual>
+    <collision>
+      <origin xyz="0 0 0" rpy="0 0 0" />
+      <geometry>
+        <mesh filename="package://deltax_descriptions/meshes/4_dof/ball_bot3_Link.STL" />
       </geometry>
     </collision>
@@ -293,12 +293,12 @@
       <origin xyz="0 0 0" rpy="0 0 0" />
       <geometry>
-        <mesh filename="package://deltax_descriptions/meshes/re2_Link.STL" />
-      </geometry>
-      <material name="LightGrey"/>
-    </visual>
-    <collision>
-      <origin xyz="0 0 0" rpy="0 0 0" />
-      <geometry>
-        <mesh filename="package://deltax_descriptions/meshes/re2_Link.STL" />
+        <mesh filename="package://deltax_descriptions/meshes/4_dof/re2_Link.STL" />
+      </geometry>
+      <material name="LightGrey"/>
+    </visual>
+    <collision>
+      <origin xyz="0 0 0" rpy="0 0 0" />
+      <geometry>
+        <mesh filename="package://deltax_descriptions/meshes/4_dof/re2_Link.STL" />
       </geometry>
     </collision>
@@ -319,12 +319,12 @@
       <origin xyz="0 0 0" rpy="0 0 0" />
       <geometry>
-        <mesh filename="package://deltax_descriptions/meshes/rf2_Link.STL" />
-      </geometry>
-      <material name="LightGrey"/>
-    </visual>
-    <collision>
-      <origin xyz="0 0 0" rpy="0 0 0" />
-      <geometry>
-        <mesh filename="package://deltax_descriptions/meshes/rf2_Link.STL" />
+        <mesh filename="package://deltax_descriptions/meshes/4_dof/rf2_Link.STL" />
+      </geometry>
+      <material name="LightGrey"/>
+    </visual>
+    <collision>
+      <origin xyz="0 0 0" rpy="0 0 0" />
+      <geometry>
+        <mesh filename="package://deltax_descriptions/meshes/4_dof/rf2_Link.STL" />
       </geometry>
     </collision>
@@ -345,12 +345,12 @@
       <origin xyz="0 0 0" rpy="0 0 0" />
       <geometry>
-        <mesh filename="package://deltax_descriptions/meshes/ball_top2_Link.STL" />
-      </geometry>
-      <material name="LightGrey"/>
-    </visual>
-    <collision>
-      <origin xyz="0 0 0" rpy="0 0 0" />
-      <geometry>
-        <mesh filename="package://deltax_descriptions/meshes/ball_top2_Link.STL" />
+        <mesh filename="package://deltax_descriptions/meshes/4_dof/ball_top2_Link.STL" />
+      </geometry>
+      <material name="LightGrey"/>
+    </visual>
+    <collision>
+      <origin xyz="0 0 0" rpy="0 0 0" />
+      <geometry>
+        <mesh filename="package://deltax_descriptions/meshes/4_dof/ball_top2_Link.STL" />
       </geometry>
     </collision>
@@ -371,12 +371,12 @@
       <origin xyz="0 0 0" rpy="0 0 0" />
       <geometry>
-        <mesh filename="package://deltax_descriptions/meshes/re3_Link.STL" />
-      </geometry>
-      <material name="LightGrey"/>
-    </visual>
-    <collision>
-      <origin xyz="0 0 0" rpy="0 0 0" />
-      <geometry>
-        <mesh filename="package://deltax_descriptions/meshes/re3_Link.STL" />
+        <mesh filename="package://deltax_descriptions/meshes/4_dof/re3_Link.STL" />
+      </geometry>
+      <material name="LightGrey"/>
+    </visual>
+    <collision>
+      <origin xyz="0 0 0" rpy="0 0 0" />
+      <geometry>
+        <mesh filename="package://deltax_descriptions/meshes/4_dof/re3_Link.STL" />
       </geometry>
     </collision>
@@ -397,12 +397,12 @@
       <origin xyz="0 0 0" rpy="0 0 0" />
       <geometry>
-        <mesh filename="package://deltax_descriptions/meshes/re4_Link.STL" />
-      </geometry>
-      <material name="LightGrey"/>
-    </visual>
-    <collision>
-      <origin xyz="0 0 0" rpy="0 0 0" />
-      <geometry>
-        <mesh filename="package://deltax_descriptions/meshes/re4_Link.STL" />
+        <mesh filename="package://deltax_descriptions/meshes/4_dof/re4_Link.STL" />
+      </geometry>
+      <material name="LightGrey"/>
+    </visual>
+    <collision>
+      <origin xyz="0 0 0" rpy="0 0 0" />
+      <geometry>
+        <mesh filename="package://deltax_descriptions/meshes/4_dof/re4_Link.STL" />
       </geometry>
     </collision>
@@ -423,5 +423,5 @@
       <origin xyz="0 0 0" rpy="0 0 0" />
       <geometry>
-        <mesh filename="package://deltax_descriptions/meshes/rf3_Link.STL" />
+        <mesh filename="package://deltax_descriptions/meshes/4_dof/rf3_Link.STL" />
       </geometry>
       <material name="LightGrey">
@@ -432,5 +432,5 @@
       <origin xyz="0 0 0" rpy="0 0 0" />
       <geometry>
-        <mesh filename="package://deltax_descriptions/meshes/rf3_Link.STL" />
+        <mesh filename="package://deltax_descriptions/meshes/4_dof/rf3_Link.STL" />
       </geometry>
     </collision>
@@ -451,12 +451,12 @@
       <origin xyz="0 0 0" rpy="0 0 0" />
       <geometry>
-        <mesh filename="package://deltax_descriptions/meshes/ball_top3_Link.STL" />
-      </geometry>
-      <material name="LightGrey"/>
-    </visual>
-    <collision>
-      <origin xyz="0 0 0" rpy="0 0 0" />
-      <geometry>
-        <mesh filename="package://deltax_descriptions/meshes/ball_top3_Link.STL" />
+        <mesh filename="package://deltax_descriptions/meshes/4_dof/ball_top3_Link.STL" />
+      </geometry>
+      <material name="LightGrey"/>
+    </visual>
+    <collision>
+      <origin xyz="0 0 0" rpy="0 0 0" />
+      <geometry>
+        <mesh filename="package://deltax_descriptions/meshes/4_dof/ball_top3_Link.STL" />
       </geometry>
     </collision>
@@ -477,12 +477,12 @@
       <origin xyz="0 0 0" rpy="0 0 0" />
       <geometry>
-        <mesh filename="package://deltax_descriptions/meshes/re5_Link.STL" />
-      </geometry>
-      <material name="LightGrey"/>
-    </visual>
-    <collision>
-      <origin xyz="0 0 0" rpy="0 0 0" />
-      <geometry>
-        <mesh filename="package://deltax_descriptions/meshes/re5_Link.STL" />
+        <mesh filename="package://deltax_descriptions/meshes/4_dof/re5_Link.STL" />
+      </geometry>
+      <material name="LightGrey"/>
+    </visual>
+    <collision>
+      <origin xyz="0 0 0" rpy="0 0 0" />
+      <geometry>
+        <mesh filename="package://deltax_descriptions/meshes/4_dof/re5_Link.STL" />
       </geometry>
     </collision>
@@ -503,12 +503,12 @@
       <origin xyz="0 0 0" rpy="0 0 0" />
       <geometry>
-        <mesh filename="package://deltax_descriptions/meshes/re6_Link.STL" />
-      </geometry>
-      <material name="LightGrey"/>
-    </visual>
-    <collision>
-      <origin xyz="0 0 0" rpy="0 0 0" />
-      <geometry>
-        <mesh filename="package://deltax_descriptions/meshes/re6_Link.STL" />
+        <mesh filename="package://deltax_descriptions/meshes/4_dof/re6_Link.STL" />
+      </geometry>
+      <material name="LightGrey"/>
+    </visual>
+    <collision>
+      <origin xyz="0 0 0" rpy="0 0 0" />
+      <geometry>
+        <mesh filename="package://deltax_descriptions/meshes/4_dof/re6_Link.STL" />
       </geometry>
     </collision>
