Commit message: joint moving joutine done!

File: deltax_descriptions/urdf/deltaxs_d800_6axis_v2.urdf.xacro (robot description, xacro)
@@ -232,5 +232,5 @@
     <parent link="axis4_Link" />
     <child link="axis5_Link" />
-    <axis xyz="0 0 1" />
+    <axis xyz="0 0 -1" />
   </joint>
   <link name="axis6_Link">

Commit message: looking good, ready for calibration!

File: deltax_descriptions/urdf/deltaxs_d800_6axis_v2.urdf.xacro (robot description, xacro)
@@ -168,5 +168,5 @@
   <link name="xyz_link">
       <visual>
-      <origin xyz="0 0 0" rpy="0 0 0" />
+      <origin xyz="0 0 0" rpy="0 0 ${pi}" />
       <geometry>
         <mesh filename="package://deltax_descriptions/meshes/6_dof/ball_moving_Link.STL" />
@@ -176,5 +176,5 @@
   </link>
   <joint name="floating_joint" type="floating">
-    <origin xyz="0 -0.034641 -0.75" rpy="0 ${pi/2} 0" />
+    <origin xyz="0 -0.034641 -0.75" rpy="0 0 ${pi/2}" />
     <parent link="base_link" />
     <child link="xyz_link" />
@@ -202,5 +202,5 @@
   </link>
   <joint name="axis4" type="continuous">
-    <origin xyz="-0.0005 0.034641 0" rpy="1.5708 -1.5562 -1.5708" />
+    <origin xyz="0.0005 -0.034641 0" rpy="1.5708 -1.5562 -1.5708" />
     <!-- <parent link="ball_moving_Link" /> -->
     <parent link="xyz_link" />

Commit message: ok going for the grasp now

File: deltax_descriptions/urdf/deltaxs_d800_6axis_v2.urdf.xacro (robot description, xacro)
@@ -176,4 +176,5 @@
   </link>
   <joint name="floating_joint" type="floating">
+  <!-- <joint name="floating_joint" type="fixed"> -->
     <origin xyz="0 -0.034641 -0.75" rpy="0 0 ${pi/2}" />
     <parent link="base_link" />

Commit message: improved hand eye routine

File: deltax_descriptions/urdf/deltaxs_d800_6axis_v2.urdf.xacro (robot description, xacro)
@@ -177,5 +177,6 @@
   <joint name="floating_joint" type="floating">
   <!-- <joint name="floating_joint" type="fixed"> -->
-    <origin xyz="0 -0.034641 -0.75" rpy="0 0 ${pi/2}" />
+    <!-- <origin xyz="0 -0.034641 -0.75" rpy="0 0 ${pi/2}" /> -->
+    <origin xyz="0 0 0" rpy="0 0 0" />
     <parent link="base_link" />
     <child link="xyz_link" />
