Commit message: direction is better but angle offsets wrong

File: deltax_descriptions/urdf/deltaxs_d800_6axis.urdf.xacro (robot description, xacro)
@@ -52,5 +52,5 @@
     <parent link="base_link" />
     <child link="rf1_Link" />
-    <axis xyz="0 0 1" />
+    <axis xyz="0 0 -1" />
   </joint>
   <link name="ball_top1_Link">
@@ -344,5 +344,5 @@
     <parent link="base_link" />
     <child link="rf2_Link" />
-    <axis xyz="0 0 1" />
+    <axis xyz="0 0 -1" />
   </joint>
   <link name="ball_top2_Link">
@@ -450,5 +450,5 @@
     <parent link="base_link" />
     <child link="rf3_Link" />
-    <axis xyz="0 0 1" />
+    <axis xyz="0 0 -1" />
   </joint>
   <link name="ball_top3_Link">

Commit message: added 4 dof meshes

File: deltax_descriptions/urdf/deltaxs_d800_6axis.urdf.xacro (robot description, xacro)
@@ -17,12 +17,12 @@
       <origin xyz="0 0 0" rpy="0 0 0" />
       <geometry>
-        <mesh filename="package://deltax_descriptions/meshes/base_link.STL" />
-      </geometry>
-      <material name="LightGrey"/>
-    </visual>
-    <collision>
-      <origin xyz="0 0 0" rpy="0 0 0" />
-      <geometry>
-        <mesh filename="package://deltax_descriptions/meshes/base_link.STL" />
+        <mesh filename="package://deltax_descriptions/meshes/6_dof/base_link.STL" />
+      </geometry>
+      <material name="LightGrey"/>
+    </visual>
+    <collision>
+      <origin xyz="0 0 0" rpy="0 0 0" />
+      <geometry>
+        <mesh filename="package://deltax_descriptions/meshes/6_dof/base_link.STL" />
       </geometry>
     </collision>
@@ -37,12 +37,12 @@
       <origin xyz="0 0 0" rpy="0 0 0" />
       <geometry>
-        <mesh filename="package://deltax_descriptions/meshes/rf1_Link.STL" />
-      </geometry>
-      <material name="LightGrey"/>
-    </visual>
-    <collision>
-      <origin xyz="0 0 0" rpy="0 0 0" />
-      <geometry>
-        <mesh filename="package://deltax_descriptions/meshes/rf1_Link.STL" />
+        <mesh filename="package://deltax_descriptions/meshes/6_dof/rf1_Link.STL" />
+      </geometry>
+      <material name="LightGrey"/>
+    </visual>
+    <collision>
+      <origin xyz="0 0 0" rpy="0 0 0" />
+      <geometry>
+        <mesh filename="package://deltax_descriptions/meshes/6_dof/rf1_Link.STL" />
       </geometry>
     </collision>
@@ -63,12 +63,12 @@
       <origin xyz="0 0 0" rpy="0 0 0" />
       <geometry>
-        <mesh filename="package://deltax_descriptions/meshes/ball_top1_Link.STL" />
-      </geometry>
-      <material name="LightGrey"/>
-    </visual>
-    <collision>
-      <origin xyz="0 0 0" rpy="0 0 0" />
-      <geometry>
-        <mesh filename="package://deltax_descriptions/meshes/ball_top1_Link.STL" />
+        <mesh filename="package://deltax_descriptions/meshes/6_dof/ball_top1_Link.STL" />
+      </geometry>
+      <material name="LightGrey"/>
+    </visual>
+    <collision>
+      <origin xyz="0 0 0" rpy="0 0 0" />
+      <geometry>
+        <mesh filename="package://deltax_descriptions/meshes/6_dof/ball_top1_Link.STL" />
       </geometry>
     </collision>
@@ -89,12 +89,12 @@
       <origin xyz="0 0 0" rpy="0 0 0" />
       <geometry>
-        <mesh filename="package://deltax_descriptions/meshes/re1_Link.STL" />
-      </geometry>
-      <material name="LightGrey"/>
-    </visual>
-    <collision>
-      <origin xyz="0 0 0" rpy="0 0 0" />
-      <geometry>
-        <mesh filename="package://deltax_descriptions/meshes/re1_Link.STL" />
+        <mesh filename="package://deltax_descriptions/meshes/6_dof/re1_Link.STL" />
+      </geometry>
+      <material name="LightGrey"/>
+    </visual>
+    <collision>
+      <origin xyz="0 0 0" rpy="0 0 0" />
+      <geometry>
+        <mesh filename="package://deltax_descriptions/meshes/6_dof/re1_Link.STL" />
       </geometry>
     </collision>
@@ -116,12 +116,12 @@
       <origin xyz="0 0 0" rpy="0 0 0" />
       <geometry>
-        <mesh filename="package://deltax_descriptions/meshes/re2_Link.STL" />
-      </geometry>
-      <material name="LightGrey"/>
-    </visual>
-    <collision>
-      <origin xyz="0 0 0" rpy="0 0 0" />
-      <geometry>
-        <mesh filename="package://deltax_descriptions/meshes/re2_Link.STL" />
+        <mesh filename="package://deltax_descriptions/meshes/6_dof/re2_Link.STL" />
+      </geometry>
+      <material name="LightGrey"/>
+    </visual>
+    <collision>
+      <origin xyz="0 0 0" rpy="0 0 0" />
+      <geometry>
+        <mesh filename="package://deltax_descriptions/meshes/6_dof/re2_Link.STL" />
       </geometry>
     </collision>
@@ -143,12 +143,12 @@
       <origin xyz="0 0 0" rpy="0 0 0" />
       <geometry>
-        <mesh filename="package://deltax_descriptions/meshes/ball_bot1_Link.STL" />
-      </geometry>
-      <material name="LightGrey"/>
-    </visual>
-    <collision>
-      <origin xyz="0 0 0" rpy="0 0 0" />
-      <geometry>
-        <mesh filename="package://deltax_descriptions/meshes/ball_bot1_Link.STL" />
+        <mesh filename="package://deltax_descriptions/meshes/6_dof/ball_bot1_Link.STL" />
+      </geometry>
+      <material name="LightGrey"/>
+    </visual>
+    <collision>
+      <origin xyz="0 0 0" rpy="0 0 0" />
+      <geometry>
+        <mesh filename="package://deltax_descriptions/meshes/6_dof/ball_bot1_Link.STL" />
       </geometry>
     </collision>
@@ -169,12 +169,12 @@
       <origin xyz="0 0 0" rpy="0 0 0" />
       <geometry>
-        <mesh filename="package://deltax_descriptions/meshes/ball_moving_Link.STL" />
-      </geometry>
-      <material name="LightGrey"/>
-    </visual>
-    <collision>
-      <origin xyz="0 0 0" rpy="0 0 0" />
-      <geometry>
-        <mesh filename="package://deltax_descriptions/meshes/ball_moving_Link.STL" />
+        <mesh filename="package://deltax_descriptions/meshes/6_dof/ball_moving_Link.STL" />
+      </geometry>
+      <material name="LightGrey"/>
+    </visual>
+    <collision>
+      <origin xyz="0 0 0" rpy="0 0 0" />
+      <geometry>
+        <mesh filename="package://deltax_descriptions/meshes/6_dof/ball_moving_Link.STL" />
       </geometry>
     </collision>
@@ -195,12 +195,12 @@
       <origin xyz="0 0 0" rpy="0 0 0" />
       <geometry>
-        <mesh filename="package://deltax_descriptions/meshes/axis4_Link.STL" />
-      </geometry>
-      <material name="LightGrey"/>
-    </visual>
-    <collision>
-      <origin xyz="0 0 0" rpy="0 0 0" />
-      <geometry>
-        <mesh filename="package://deltax_descriptions/meshes/axis4_Link.STL" />
+        <mesh filename="package://deltax_descriptions/meshes/6_dof/axis4_Link.STL" />
+      </geometry>
+      <material name="LightGrey"/>
+    </visual>
+    <collision>
+      <origin xyz="0 0 0" rpy="0 0 0" />
+      <geometry>
+        <mesh filename="package://deltax_descriptions/meshes/6_dof/axis4_Link.STL" />
       </geometry>
     </collision>
@@ -221,12 +221,12 @@
       <origin xyz="0 0 0" rpy="0 0 0" />
       <geometry>
-        <mesh filename="package://deltax_descriptions/meshes/axis5_Link.STL" />
-      </geometry>
-      <material name="LightGrey"/>
-    </visual>
-    <collision>
-      <origin xyz="0 0 0" rpy="0 0 0" />
-      <geometry>
-        <mesh filename="package://deltax_descriptions/meshes/axis5_Link.STL" />
+        <mesh filename="package://deltax_descriptions/meshes/6_dof/axis5_Link.STL" />
+      </geometry>
+      <material name="LightGrey"/>
+    </visual>
+    <collision>
+      <origin xyz="0 0 0" rpy="0 0 0" />
+      <geometry>
+        <mesh filename="package://deltax_descriptions/meshes/6_dof/axis5_Link.STL" />
       </geometry>
     </collision>
@@ -247,12 +247,12 @@
       <origin xyz="0 0 0" rpy="0 0 0" />
       <geometry>
-        <mesh filename="package://deltax_descriptions/meshes/axis6_Link.STL" />
-      </geometry>
-      <material name="LightGrey"/>
-    </visual>
-    <collision>
-      <origin xyz="0 0 0" rpy="0 0 0" />
-      <geometry>
-        <mesh filename="package://deltax_descriptions/meshes/axis6_Link.STL" />
+        <mesh filename="package://deltax_descriptions/meshes/6_dof/axis6_Link.STL" />
+      </geometry>
+      <material name="LightGrey"/>
+    </visual>
+    <collision>
+      <origin xyz="0 0 0" rpy="0 0 0" />
+      <geometry>
+        <mesh filename="package://deltax_descriptions/meshes/6_dof/axis6_Link.STL" />
       </geometry>
     </collision>
@@ -275,12 +275,12 @@
       <origin xyz="0 0 0" rpy="0 0 0" />
       <geometry>
-        <mesh filename="package://deltax_descriptions/meshes/ball_bot2_Link.STL" />
-      </geometry>
-      <material name="LightGrey"/>
-    </visual>
-    <collision>
-      <origin xyz="0 0 0" rpy="0 0 0" />
-      <geometry>
-        <mesh filename="package://deltax_descriptions/meshes/ball_bot2_Link.STL" />
+        <mesh filename="package://deltax_descriptions/meshes/6_dof/ball_bot2_Link.STL" />
+      </geometry>
+      <material name="LightGrey"/>
+    </visual>
+    <collision>
+      <origin xyz="0 0 0" rpy="0 0 0" />
+      <geometry>
+        <mesh filename="package://deltax_descriptions/meshes/6_dof/ball_bot2_Link.STL" />
       </geometry>
     </collision>
@@ -301,12 +301,12 @@
       <origin xyz="0 0 0" rpy="0 0 0" />
       <geometry>
-        <mesh filename="package://deltax_descriptions/meshes/ball_bot3_Link.STL" />
-      </geometry>
-      <material name="LightGrey"/>
-    </visual>
-    <collision>
-      <origin xyz="0 0 0" rpy="0 0 0" />
-      <geometry>
-        <mesh filename="package://deltax_descriptions/meshes/ball_bot3_Link.STL" />
+        <mesh filename="package://deltax_descriptions/meshes/6_dof/ball_bot3_Link.STL" />
+      </geometry>
+      <material name="LightGrey"/>
+    </visual>
+    <collision>
+      <origin xyz="0 0 0" rpy="0 0 0" />
+      <geometry>
+        <mesh filename="package://deltax_descriptions/meshes/6_dof/ball_bot3_Link.STL" />
       </geometry>
     </collision>
@@ -329,12 +329,12 @@
       <origin xyz="0 0 0" rpy="0 0 0" />
       <geometry>
-        <mesh filename="package://deltax_descriptions/meshes/rf2_Link.STL" />
-      </geometry>
-      <material name="LightGrey"/>
-    </visual>
-    <collision>
-      <origin xyz="0 0 0" rpy="0 0 0" />
-      <geometry>
-        <mesh filename="package://deltax_descriptions/meshes/rf2_Link.STL" />
+        <mesh filename="package://deltax_descriptions/meshes/6_dof/rf2_Link.STL" />
+      </geometry>
+      <material name="LightGrey"/>
+    </visual>
+    <collision>
+      <origin xyz="0 0 0" rpy="0 0 0" />
+      <geometry>
+        <mesh filename="package://deltax_descriptions/meshes/6_dof/rf2_Link.STL" />
       </geometry>
     </collision>
@@ -355,12 +355,12 @@
       <origin xyz="0 0 0" rpy="0 0 0" />
       <geometry>
-        <mesh filename="package://deltax_descriptions/meshes/ball_top2_Link.STL" />
-      </geometry>
-      <material name="LightGrey"/>
-    </visual>
-    <collision>
-      <origin xyz="0 0 0" rpy="0 0 0" />
-      <geometry>
-        <mesh filename="package://deltax_descriptions/meshes/ball_top2_Link.STL" />
+        <mesh filename="package://deltax_descriptions/meshes/6_dof/ball_top2_Link.STL" />
+      </geometry>
+      <material name="LightGrey"/>
+    </visual>
+    <collision>
+      <origin xyz="0 0 0" rpy="0 0 0" />
+      <geometry>
+        <mesh filename="package://deltax_descriptions/meshes/6_dof/ball_top2_Link.STL" />
       </geometry>
     </collision>
@@ -381,12 +381,12 @@
       <origin xyz="0 0 0" rpy="0 0 0" />
       <geometry>
-        <mesh filename="package://deltax_descriptions/meshes/re3_Link.STL" />
-      </geometry>
-      <material name="LightGrey"/>
-    </visual>
-    <collision>
-      <origin xyz="0 0 0" rpy="0 0 0" />
-      <geometry>
-        <mesh filename="package://deltax_descriptions/meshes/re3_Link.STL" />
+        <mesh filename="package://deltax_descriptions/meshes/6_dof/re3_Link.STL" />
+      </geometry>
+      <material name="LightGrey"/>
+    </visual>
+    <collision>
+      <origin xyz="0 0 0" rpy="0 0 0" />
+      <geometry>
+        <mesh filename="package://deltax_descriptions/meshes/6_dof/re3_Link.STL" />
       </geometry>
     </collision>
@@ -407,12 +407,12 @@
       <origin xyz="0 0 0" rpy="0 0 0" />
       <geometry>
-        <mesh filename="package://deltax_descriptions/meshes/re4_Link.STL" />
-      </geometry>
-      <material name="LightGrey"/>
-    </visual>
-    <collision>
-      <origin xyz="0 0 0" rpy="0 0 0" />
-      <geometry>
-        <mesh filename="package://deltax_descriptions/meshes/re4_Link.STL" />
+        <mesh filename="package://deltax_descriptions/meshes/6_dof/re4_Link.STL" />
+      </geometry>
+      <material name="LightGrey"/>
+    </visual>
+    <collision>
+      <origin xyz="0 0 0" rpy="0 0 0" />
+      <geometry>
+        <mesh filename="package://deltax_descriptions/meshes/6_dof/re4_Link.STL" />
       </geometry>
     </collision>
@@ -435,12 +435,12 @@
       <origin xyz="0 0 0" rpy="0 0 0" />
       <geometry>
-        <mesh filename="package://deltax_descriptions/meshes/rf3_Link.STL" />
-      </geometry>
-      <material name="LightGrey"/>
-    </visual>
-    <collision>
-      <origin xyz="0 0 0" rpy="0 0 0" />
-      <geometry>
-        <mesh filename="package://deltax_descriptions/meshes/rf3_Link.STL" />
+        <mesh filename="package://deltax_descriptions/meshes/6_dof/rf3_Link.STL" />
+      </geometry>
+      <material name="LightGrey"/>
+    </visual>
+    <collision>
+      <origin xyz="0 0 0" rpy="0 0 0" />
+      <geometry>
+        <mesh filename="package://deltax_descriptions/meshes/6_dof/rf3_Link.STL" />
       </geometry>
     </collision>
@@ -461,12 +461,12 @@
       <origin xyz="0 0 0" rpy="0 0 0" />
       <geometry>
-        <mesh filename="package://deltax_descriptions/meshes/ball_top3_Link.STL" />
-      </geometry>
-      <material name="LightGrey"/>
-    </visual>
-    <collision>
-      <origin xyz="0 0 0" rpy="0 0 0" />
-      <geometry>
-        <mesh filename="package://deltax_descriptions/meshes/ball_top3_Link.STL" />
+        <mesh filename="package://deltax_descriptions/meshes/6_dof/ball_top3_Link.STL" />
+      </geometry>
+      <material name="LightGrey"/>
+    </visual>
+    <collision>
+      <origin xyz="0 0 0" rpy="0 0 0" />
+      <geometry>
+        <mesh filename="package://deltax_descriptions/meshes/6_dof/ball_top3_Link.STL" />
       </geometry>
     </collision>
@@ -487,12 +487,12 @@
       <origin xyz="0 0 0" rpy="0 0 0" />
       <geometry>
-        <mesh filename="package://deltax_descriptions/meshes/re5_Link.STL" />
-      </geometry>
-      <material name="LightGrey"/>
-    </visual>
-    <collision>
-      <origin xyz="0 0 0" rpy="0 0 0" />
-      <geometry>
-        <mesh filename="package://deltax_descriptions/meshes/re5_Link.STL" />
+        <mesh filename="package://deltax_descriptions/meshes/6_dof/re5_Link.STL" />
+      </geometry>
+      <material name="LightGrey"/>
+    </visual>
+    <collision>
+      <origin xyz="0 0 0" rpy="0 0 0" />
+      <geometry>
+        <mesh filename="package://deltax_descriptions/meshes/6_dof/re5_Link.STL" />
       </geometry>
     </collision>
@@ -513,12 +513,12 @@
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
File: deltax_descriptions/urdf/deltaxs_v4_d800.urdf (robot description, URDF)
Before this commit: robot deltax_descriptions, 17 links, 16 joints
Links:
- link ball_bot1_Link: geometry collision mesh filename=package://deltax_descriptions/meshes/4_dof/ball_bot1_Link.S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; visual mesh filename=package://deltax_descriptions/meshes/4_dof/ball_bot1_Link.S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
- link ball_bot2_Link: geometry collision mesh filename=package://deltax_descriptions/meshes/4_dof/ball_bot2_Link.S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; visual mesh filename=package://deltax_descriptions/meshes/4_dof/ball_bot2_Link.S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
- link ball_bot3_Link: geometry collision mesh filename=package://deltax_descriptions/meshes/4_dof/ball_bot3_Link.S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; visual mesh filename=package://deltax_descriptions/meshes/4_dof/ball_bot3_Link.S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
- link ball_moving_Link: geometry collision mesh filename=package://deltax_descriptions/meshes/4_dof/ball_moving_Link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; visual mesh filename=package://deltax_descriptions/meshes/4_dof/ball_moving_Link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
- link ball_top1_Link: geometry collision mesh filename=package://deltax_descriptions/meshes/4_dof/ball_top1_Link.S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; visual mesh filename=package://deltax_descriptions/meshes/4_dof/ball_top1_Link.S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
- link ball_top2_Link: geometry collision mesh filename=package://deltax_descriptions/meshes/4_dof/ball_top2_Link.S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; visual mesh filename=package://deltax_descriptions/meshes/4_dof/ball_top2_Link.S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
- link ball_top3_Link: geometry collision mesh filename=package://deltax_descriptions/meshes/4_dof/ball_top3_Link.S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; visual mesh filename=package://deltax_descriptions/meshes/4_dof/ball_top3_Link.S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
- link base_link: geometry collision mesh filename=package://deltax_descriptions/meshes/4_dof/base_link.STL; visual mesh filename=package://deltax_descriptions/meshes/4_dof/base_link.STL
- link re1_Link: geometry collision mesh filename=package://deltax_descriptions/meshes/4_dof/re1_Link.STL; visual mesh filename=package://deltax_descriptions/meshes/4_dof/re1_Link.STL
- link re2_Link: geometry collision mesh filename=package://deltax_descriptions/meshes/4_dof/re2_Link.STL; visual mesh filename=package://deltax_descriptions/meshes/4_dof/re2_Link.STL
- link re3_Link: geometry collision mesh filename=package://deltax_descriptions/meshes/4_dof/re3_Link.STL; visual mesh filename=package://deltax_descriptions/meshes/4_dof/re3_Link.STL
- link re4_Link: geometry collision mesh filename=package://deltax_descriptions/meshes/4_dof/re4_Link.STL; visual mesh filename=package://deltax_descriptions/meshes/4_dof/re4_Link.STL
- link re5_Link: geometry collision mesh filename=package://deltax_descriptions/meshes/4_dof/re5_Link.STL; visual mesh filename=package://deltax_descriptions/meshes/4_dof/re5_Link.STL
- link re6_Link: geometry collision mesh filename=package://deltax_descriptions/meshes/4_dof/re6_Link.STL; visual mesh filename=package://deltax_descriptions/meshes/4_dof/re6_Link.STL
- link rf1_Link: geometry collision mesh filename=package://deltax_descriptions/meshes/4_dof/rf1_Link.STL; visual mesh filename=package://deltax_descriptions/meshes/4_dof/rf1_Link.STL
- link rf2_Link: geometry collision mesh filename=package://deltax_descriptions/meshes/4_dof/rf2_Link.STL; visual mesh filename=package://deltax_descriptions/meshes/4_dof/rf2_Link.STL
- link rf3_Link: geometry collision mesh filename=package://deltax_descriptions/meshes/4_dof/rf3_Link.STL; visual mesh filename=package://deltax_descriptions/meshes/4_dof/rf3_Link.STL

Commit message: pivoting to 4 DOF robot

File: deltax_descriptions/urdf/deltaxs_d800_6axis.urdf.xacro (robot description, xacro)
@@ -179,5 +179,5 @@
       </geometry>
     </collision>
-  </link>
+  </link>l
   <joint name="ball_moving" type="continuous">
     <origin xyz="0 0.033373 0" rpy="-1.5708 -0.58245 0" />
