Commit message: reformatting project dir

File: deltax_descriptions/urdf/deltaxs_d800_4axis_v1.urdf.xacro (robot description, xacro)
@@ -175,7 +175,7 @@
     </visual>
   </link>
-  <!-- <joint name="floating_joint" type="floating"> -->
-  <joint name="floating_joint" type="fixed">
-    <origin xyz="0 -0.034641 -0.805" rpy="0 0 0" />
+  <joint name="floating_joint" type="floating">
+  <!-- <joint name="floating_joint" type="fixed"> -->
+    <!-- <origin xyz="0 -0.034641 -0.805" rpy="0 0 0" /> -->
     <origin xyz="0 0 0" rpy="0 0 0" />
     <parent link="base_link" />
