Commit message: good enough IK for now

File: deltax_descriptions/urdf/deltaxs_d800_4axis_v2.urdf.xacro (robot description, xacro)
@@ -199,6 +199,7 @@
     </collision>
   </link>
+  <!-- rotate this to set the zero properly... -->
   <joint name="axis4" type="continuous">
-    <origin xyz="0 0 0.0005" rpy="0 0 ${pi/2}" />
+    <origin xyz="0 0 0.0005" rpy="0 0 0" />
     <parent link="xyz_link" />
     <child link="axis4_Link" />
